File: KiCad-Shield-Led/KiCad-Shield-Led.sch (KiCad schematic (older format))
At the start: 16 parts, among them P1 Power, P2 Analog, P3 Digital, P4 Digital, P5 CONN_01X01, P6 CONN_01X01, P7 CONN_01X01, P8 CONN_01X01

Commit message: Generation de la netlist
Parts:
- D1, D2, D3, D4: footprint (none) -> LED_THT:LED_D5.0mm
- R1, R2, R3, R4: footprint (none) -> Resistor_THT:R_Axial_DIN0207_L6.3mm_D2.5mm_P10.16mm_Horizontal
Changed lines of the file:
@@
 F 0 "D1" V 5689 2632 50  0000 R CNN
 F 1 "LED" V 5598 2632 50  0000 R CNN
-F 2 "" H 5650 2750 50  0001 C CNN
+F 2 "LED_THT:LED_D5.0mm" H 5650 2750 50  0001 C CNN
 F 3 "~" H 5650 2750 50  0001 C CNN
 	1    5650 2750
@@
 F 0 "R1" H 5720 2396 50  0000 L CNN
 F 1 "470" H 5720 2305 50  0000 L CNN
-F 2 "" V 5580 2350 50  0001 C CNN
+F 2 "Resistor_THT:R_Axial_DIN0207_L6.3mm_D2.5mm_P10.16mm_Horizontal" V 5580 2350 50  0001 C CNN
 F 3 "~" H 5650 2350 50  0001 C CNN
 	1    5650 2350
@@
 F 0 "D2" V 6039 2632 50  0000 R CNN
 F 1 "LED" V 5948 2632 50  0000 R CNN
-F 2 "" H 6000 2750 50  0001 C CNN
+F 2 "LED_THT:LED_D5.0mm" H 6000 2750 50  0001 C CNN
 F 3 "~" H 6000 2750 50  0001 C CNN
 	1    6000 2750
@@
 F 0 "R2" H 6070 2396 50  0000 L CNN
 F 1 "470" H 6070 2305 50  0000 L CNN
-F 2 "" V 5930 2350 50  0001 C CNN
+F 2 "Resistor_THT:R_Axial_DIN0207_L6.3mm_D2.5mm_P10.16mm_Horizontal" V 5930 2350 50  0001 C CNN
 F 3 "~" H 6000 2350 50  0001 C CNN
 	1    6000 2350
@@
 F 0 "D3" V 6389 2632 50  0000 R CNN
 F 1 "LED" V 6298 2632 50  0000 R CNN
-F 2 "" H 6350 2750 50  0001 C CNN
+F 2 "LED_THT:LED_D5.0mm" H 6350 2750 50  0001 C CNN
 F 3 "~" H 6350 2750 50  0001 C CNN
 	1    6350 2750
@@
 F 0 "R3" H 6420 2396 50  0000 L CNN
 F 1 "470" H 6420 2305 50  0000 L CNN
-F 2 "" V 6280 2350 50  0001 C CNN
+F 2 "Resistor_THT:R_Axial_DIN0207_L6.3mm_D2.5mm_P10.16mm_Horizontal" V 6280 2350 50  0001 C CNN
 F 3 "~" H 6350 2350 50  0001 C CNN
 	1    6350 2350
@@
 F 0 "D4" V 6739 2632 50  0000 R CNN
 F 1 "LED" V 6648 2632 50  0000 R CNN
-F 2 "" H 6700 2750 50  0001 C CNN
+F 2 "LED_THT:LED_D5.0mm" H 6700 2750 50  0001 C CNN
 F 3 "~" H 6700 2750 50  0001 C CNN
 	1    6700 2750
@@
 F 0 "R4" H 6770 2396 50  0000 L CNN
 F 1 "470" H 6770 2305 50  0000 L CNN
-F 2 "" V 6630 2350 50  0001 C CNN
+F 2 "Resistor_THT:R_Axial_DIN0207_L6.3mm_D2.5mm_P10.16mm_Horizontal" V 6630 2350 50  0001 C CNN
 F 3 "~" H 6700 2350 50  0001 C CNN
 	1    6700 2350

Commit message: Place components
Other:
- moved on the sheet: D1, D2, D3, D4, R1, R2, R3, R4
Changed lines of the file:
@@
 L Device:LED D1
 U 1 1 5FC4CFF8
-P 5650 2750
-F 0 "D1" V 5689 2632 50  0000 R CNN
-F 1 "LED" V 5598 2632 50  0000 R CNN
-F 2 "LED_THT:LED_D5.0mm" H 5650 2750 50  0001 C CNN
-F 3 "~" H 5650 2750 50  0001 C CNN
-	1    5650 2750
+P 6550 2650
+F 0 "D1" V 6589 2532 50  0000 R CNN
+F 1 "LED" V 6498 2532 50  0000 R CNN
+F 2 "LED_THT:LED_D5.0mm" H 6550 2650 50  0001 C CNN
+F 3 "~" H 6550 2650 50  0001 C CNN
+	1    6550 2650
 	0    -1   -1   0
 $EndComp
@@
 L Device:R R1
 U 1 1 5FC4E899
-P 5650 2350
-F 0 "R1" H 5720 2396 50  0000 L CNN
-F 1 "470" H 5720 2305 50  0000 L CNN
-F 2 "Resistor_THT:R_Axial_DIN0207_L6.3mm_D2.5mm_P10.16mm_Horizontal" V 5580 2350 50  0001 C CNN
-F 3 "~" H 5650 2350 50  0001 C CNN
-	1    5650 2350
+P 6550 2250
+F 0 "R1" H 6620 2296 50  0000 L CNN
+F 1 "470" H 6620 2205 50  0000 L CNN
+F 2 "Resistor_THT:R_Axial_DIN0207_L6.3mm_D2.5mm_P10.16mm_Horizontal" V 6480 2250 50  0001 C CNN
+F 3 "~" H 6550 2250 50  0001 C CNN
+	1    6550 2250
 	1    0    0    -1
 $EndComp
 Wire Wire Line
-	5650 2500 5650 2600
+	6550 2400 6550 2500
 Wire Wire Line
-	5650 2900 5650 3150
+	6550 2800 6550 3050
 Wire Wire Line
-	5650 3150 6000 3150
+	6550 3050 6900 3050
 Wire Wire Line
-	7100 3150 7100 3250
+	8000 3050 8000 3150
 $Comp
 L Device:LED D2
 U 1 1 5FC5721B
-P 6000 2750
-F 0 "D2" V 6039 2632 50  0000 R CNN
-F 1 "LED" V 5948 2632 50  0000 R CNN
-F 2 "LED_THT:LED_D5.0mm" H 6000 2750 50  0001 C CNN
-F 3 "~" H 6000 2750 50  0001 C CNN
-	1    6000 2750
+P 6900 2650
+F 0 "D2" V 6939 2532 50  0000 R CNN
+F 1 "LED" V 6848 2532 50  0000 R CNN
+F 2 "LED_THT:LED_D5.0mm" H 6900 2650 50  0001 C CNN
+F 3 "~" H 6900 2650 50  0001 C CNN
+	1    6900 2650
 	0    -1   -1   0
 $EndComp
@@
 L Device:R R2
 U 1 1 5FC5738B
-P 6000 2350
-F 0 "R2" H 6070 2396 50  0000 L CNN
-F 1 "470" H 6070 2305 50  0000 L CNN
-F 2 "Resistor_THT:R_Axial_DIN0207_L6.3mm_D2.5mm_P10.16mm_Horizontal" V 5930 2350 50  0001 C CNN
-F 3 "~" H 6000 2350 50  0001 C CNN
-	1    6000 2350
+P 6900 2250
+F 0 "R2" H 6970 2296 50  0000 L CNN
+F 1 "470" H 6970 2205 50  0000 L CNN
+F 2 "Resistor_THT:R_Axial_DIN0207_L6.3mm_D2.5mm_P10.16mm_Horizontal" V 6830 2250 50  0001 C CNN
+F 3 "~" H 6900 2250 50  0001 C CNN
+	1    6900 2250
 	1    0    0    -1
 $EndComp
 Wire Wire Line
-	6000 2500 6000 2600
+	6900 2400 6900 2500
 Wire Wire Line
-	6000 2900 6000 3150
-Connection ~ 6000 3150
+	6900 2800 6900 3050
+Connection ~ 6900 3050
 Wire Wire Line
-	6000 3150 6350 3150
+	6900 3050 7250 3050
 $Comp
 L Device:LED D3
 U 1 1 5FC5A1AB
-P 6350 2750
-F 0 "D3" V 6389 2632 50  0000 R CNN
-F 1 "LED" V 6298 2632 50  0000 R CNN
-F 2 "LED_THT:LED_D5.0mm" H 6350 2750 50  0001 C CNN
-F 3 "~" H 6350 2750 50  0001 C CNN
-	1    6350 2750
+P 7250 2650
+F 0 "D3" V 7289 2532 50  0000 R CNN
+F 1 "LED" V 7198 2532 50  0000 R CNN
+F 2 "LED_THT:LED_D5.0mm" H 7250 2650 50  0001 C CNN
+F 3 "~" H 7250 2650 50  0001 C CNN
+	1    7250 2650
 	0    -1   -1   0
 $EndComp
@@
 L Device:R R3
 U 1 1 5FC5A343
-P 6350 2350
-F 0 "R3" H 6420 2396 50  0000 L CNN
-F 1 "470" H 6420 2305 50  0000 L CNN
-F 2 "Resistor_THT:R_Axial_DIN0207_L6.3mm_D2.5mm_P10.16mm_Horizontal" V 6280 2350 50  0001 C CNN
-F 3 "~" H 6350 2350 50  0001 C CNN
-	1    6350 2350
+P 7250 2250
+F 0 "R3" H 7320 2296 50  0000 L CNN
+F 1 "470" H 7320 2205 50  0000 L CNN
+F 2 "Resistor_THT:R_Axial_DIN0207_L6.3mm_D2.5mm_P10.16mm_Horizontal" V 7180 2250 50  0001 C CNN
+F 3 "~" H 7250 2250 50  0001 C CNN
+	1    7250 2250
 	1    0    0    -1
 $EndComp
 Wire Wire Line
-	6350 2500 6350 2600
+	7250 2400 7250 2500
 Wire Wire Line
-	6350 2900 6350 3150
+	7250 2800 7250 3050
 $Comp
 L Device:LED D4
 U 1 1 5FC5A34F
-P 6700 2750
-F 0 "D4" V 6739 2632 50  0000 R CNN
-F 1 "LED" V 6648 2632 50  0000 R CNN
-F 2 "LED_THT:LED_D5.0mm" H 6700 2750 50  0001 C CNN
-F 3 "~" H 6700 2750 50  0001 C CNN
-	1    6700 2750
+P 7600 2650
+F 0 "D4" V 7639 2532 50  0000 R CNN
+F 1 "LED" V 7548 2532 50  0000 R CNN
+F 2 "LED_THT:LED_D5.0mm" H 7600 2650 50  0001 C CNN
+F 3 "~" H 7600 2650 50  0001 C CNN
+	1    7600 2650
 	0    -1   -1   0
 $EndComp
@@
 L Device:R R4
 U 1 1 5FC5A359
-P 6700 2350
-F 0 "R4" H 6770 2396 50  0000 L CNN
-F 1 "470" H 6770 2305 50  0000 L CNN
-F 2 "Resistor_THT:R_Axial_DIN0207_L6.3mm_D2.5mm_P10.16mm_Horizontal" V 6630 2350 50  0001 C CNN
-F 3 "~" H 6700 2350 50  0001 C CNN
-	1    6700 2350
+P 7600 2250
+F 0 "R4" H 7670 2296 50  0000 L CNN
+F 1 "470" H 7670 2205 50  0000 L CNN
+F 2 "Resistor_THT:R_Axial_DIN0207_L6.3mm_D2.5mm_P10.16mm_Horizontal" V 7530 2250 50  0001 C CNN
+F 3 "~" H 7600 2250 50  0001 C CNN
+	1    7600 2250
 	1    0    0    -1
 $EndComp
 Wire Wire Line
-	6700 2500 6700 2600
+	7600 2400 7600 2500
 Wire Wire Line
-	6700 2900 6700 3150
-Connection ~ 6350 3150
+	7600 2800 7600 3050
+Connection ~ 7250 3050
 Wire Wire Line
-	6350 3150 6700 3150
-Connection ~ 6700 3150
+	7250 3050 7600 3050
+Connection ~ 7600 3050
 Wire Wire Line
-	6700 3150 7100 3150
+	7600 3050 8000 3050
 $Comp
 L power:GND #PWR05
 U 1 1 5FC5CA17
-P 7100 3250
-F 0 "#PWR05" H 7100 3000 50  0001 C CNN
-F 1 "GND" H 7105 3077 50  0000 C CNN
-F 2 "" H 7100 3250 50  0001 C CNN
-F 3 "" H 7100 3250 50  0001 C CNN
-	1    7100 3250
+P 8000 3150
+F 0 "#PWR05" H 8000 2900 50  0001 C CNN
+F 1 "GND" H 8005 2977 50  0000 C CNN
+F 2 "" H 8000 3150 50  0001 C CNN
+F 3 "" H 8000 3150 50  0001 C CNN
+	1    8000 3150
 	1    0    0    -1
 $EndComp
 Wire Wire Line
-	6700 2200 6700 2100
+	7600 2100 7600 2000
 Wire Wire Line
-	6700 2100 7050 2100
+	7600 2000 7950 2000
 Wire Wire Line
-	6350 2200 6350 2000
+	7250 2100 7250 1900
 Wire Wire Line
-	6350 2000 7050 2000
+	7250 1900 7950 1900
 Wire Wire Line
-	6000 1900 7050 1900
+	6900 1800 7950 1800
 Wire Wire Line
-	6000 1900 6000 2200
+	6900 1800 6900 2100
 Wire Wire Line
-	5650 2200 5650 1800
+	6550 2100 6550 1700
 Wire Wire Line
-	5650 1800 7050 1800
-Text Label 7050 1800 0    50   ~ 0
+	6550 1700 7950 1700
+Text Label 7950 1700 0    50   ~ 0
 LED1
-Text Label 7050 1900 0    50   ~ 0
+Text Label 7950 1800 0    50   ~ 0
 LED2
-Text Label 7050 2000 0    50   ~ 0
+Text Label 7950 1900 0    50   ~ 0
 LED3
-Text Label 7050 2100 0    50   ~ 0
+Text Label 7950 2000 0    50   ~ 0
 LED4
 Text Label 10550 1700 0    50   ~ 0
